Commit message: Patch official repo with new splat + fix wrist camera lag

File: splatsim/robot_definitions/urdf/sisbot.urdf (robot description, URDF)
Before this commit: robot sisbot, 21 links, 20 joints
Links:
- removed link dummy_center_indicator_link
- added link wrist_camera_link; collision box size=0.072 0.051 0.034; visual box size=0.072 0.051 0.034
- added link wrist_camera_vis_x_link; visual cylinder length=0.1 radius=0.005
- added link wrist_camera_vis_y_link; visual cylinder length=0.1 radius=0.005
- added link wrist_camera_vis_z_link; visual cylinder length=0.1 radius=0.005
Joints:
- removed joint dummy_center_fixed_joint
- added joint wrist_camera_vis_joint: type fixed, parent robotiq_arg2f_base_link, child wrist_camera_link, origin xyz=-0.1 0 -0.0 rpy=0 0 -1.57
- added joint wrist_camera_vis_x_joint: type fixed, parent wrist_camera_link, child wrist_camera_vis_x_link, origin xyz=0 0 0 rpy=0 0 0
- added joint wrist_camera_vis_y_joint: type fixed, parent wrist_camera_link, child wrist_camera_vis_y_link, origin xyz=0 0 0 rpy=0 0 0
- added joint wrist_camera_vis_z_joint: type fixed, parent wrist_camera_link, child wrist_camera_vis_z_link, origin xyz=0 0 0 rpy=0 0 0
